File: ergogen/board.kicad_pcb (KiCad board)
At the start: 2 copper layers, 154.2 x 107.9 mm, 58 parts

Commit message: ok looking good
Parts:
- turned D1 to 196 degrees
- turned D10 to 184 degrees
- turned D11 to 184 degrees
- turned D12 to 184 degrees
- turned D13 to 180 degrees
- turned D14 to 180 degrees
- turned D15 to 180 degrees
- turned D16 to 180 degrees
- turned D17 to 180 degrees
- turned D18 to 180 degrees
- turned D19 to 184 degrees
- turned D2 to 196 degrees
- turned D20 to 174 degrees
- turned D21 to 164 degrees
- turned D22 to 154 degrees
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