File: ergogen/output/pcbs/board.kicad_pcb (KiCad board)
At the start: 2 copper layers, 155.7 x 107.9 mm, 58 parts

Commit message: pretty sweet
Routing:
- net BAT_P: track 0.00 -> 2.00 mm, vias 0 -> 1
Changed lines of the file:
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@@
         (pad "11" thru_hole oval (at -1 0 90) (size 1.2 1.75) (drill 0.75) (layers "*.Cu" "*.Mask") (net 81 "JST1_1"))
         (pad "12" thru_hole oval (at 1 0 90) (size 1.2 1.75) (drill 0.75) (layers "*.Cu" "*.Mask") (net 82 "JST1_2"))
-        (pad "21" smd custom (at -1 1.8 270) (size 0.1 0.1) (layers "F.Cu" "F.Mask" "F.Paste")
-            (clearance 0.1) (zone_connect 0)
-            (options (clearance outline) (anchor rect))
-            (primitives
-                (gr_poly
-                    (pts
-                        (xy 0.6 0.4)
-                        (xy -0.6 0.4)
-                        (xy -0.6 0.2)
-                        (xy 0 -0.4)
-                        (xy 0.6 0.2)
-                    )
-                    (width 0)
-                    (fill yes)
-                )
-            )
-            (net 81 "JST1_1")
-        )
-        (pad "31" smd custom (at -1 1.8 270) (size 0.1 0.1) (layers "B.Cu" "B.Mask" "B.Paste")
-            (clearance 0.1) (zone_connect 0)
-            (options (clearance outline) (anchor rect))
-            (primitives
-                (gr_poly
-                    (pts
-                        (xy 0.6 0.4)
-                        (xy -0.6 0.4)
-                        (xy -0.6 0.2)
-                        (xy 0 -0.4)
-                        (xy 0.6 0.2)
-                    )
-                    (width 0)
-                    (fill yes)
-                )
-            )
-            (net 81 "JST1_1")
-        )
-        (pad "22" smd custom (at 1 1.8 270) (size 0.1 0.1) (layers "F.Cu" "F.Mask" "F.Paste")
-            (clearance 0.1) (zone_connect 0)
-            (options (clearance outline) (anchor rect))
-            (primitives
-                (gr_poly
-                    (pts
-                        (xy 0.6 0.4)
-                        (xy -0.6 0.4)
-                        (xy -0.6 0.2)
-                        (xy 0 -0.4)
-                        (xy 0.6 0.2)
-                    )
-                    (width 0)
-                    (fill yes)
-                )
-            )
-            (net 82 "JST1_2")
-        )
-        (pad "32" smd custom (at 1 1.8 270) (size 0.1 0.1) (layers "B.Cu" "B.Mask" "B.Paste")
-            (clearance 0.1) (zone_connect 0)
-            (options (clearance outline) (anchor rect))
-            (primitives
-                (gr_poly
-                    (pts
-                        (xy 0.6 0.4)
-                        (xy -0.6 0.4)
-                        (xy -0.6 0.2)
-                        (xy 0 -0.4)
-                        (xy 0.6 0.2)
-                    )
-                    (width 0)
-                    (fill yes)
-                )
-            )
-            (net 82 "JST1_2")
-        )
-        (pad "1" smd custom (at -1 2.816 270) (size 1.2 0.5) (layers "F.Cu" "F.Mask" "F.Paste") (net 80 "BAT_P")
-            (clearance 0.1) (zone_connect 0)
-            (options (clearance outline) (anchor rect))
-            (primitives
-                (gr_poly
-                    (pts
-                        (xy 0.6 0)
-                        (xy -0.6 0)
-                        (xy -0.6 1)
-                        (xy 0 0.4)
-                        (xy 0.6 1)
-                    )
-                    (width 0)
-                    (fill yes)
-                )
-            )
-        )
-        (pad "1" smd custom (at 1 2.816 270) (size 1.2 0.5) (layers "B.Cu" "B.Mask" "B.Paste") (net 80 "BAT_P")
-            (clearance 0.1) (zone_connect 0)
-            (options (clearance outline) (anchor rect))
-            (primitives
-                (gr_poly
-                    (pts
-                        (xy 0.6 0)
-                        (xy -0.6 0)
-                        (xy -0.6 1)
-                        (xy 0 0.4)
-                        (xy 0.6 1)
-                    )
-                    (width 0)
-                    (fill yes)
-                )
-            )
-        )
-        (pad "2" smd custom (at -1 2.816 270) (size 1.2 0.5) (layers "B.Cu" "B.Mask" "B.Paste") (net 3 "GND")
-            (clearance 0.1) (zone_connect 0)
-            (options (clearance outline) (anchor rect))
-            (primitives
-                (gr_poly
-                    (pts
-                        (xy 0.6 0)
-                        (xy -0.6 0)
-                        (xy -0.6 1)
-                        (xy 0 0.4)
-                        (xy 0.6 1)
-                    )
-                    (width 0)
-                    (fill yes)
-                )
-            )
-        )
-        (pad "2" smd custom (at 1 2.816 270) (size 1.2 0.5) (layers "F.Cu" "F.Mask" "F.Paste") (net 3 "GND")
-            (clearance 0.1) (zone_connect 0)
-            (options (clearance outline) (anchor rect))
-            (primitives
-                (gr_poly
-                    (pts
-                        (xy 0.6 0)
-                        (xy -0.6 0)
-                        (xy -0.6 1)
-                        (xy 0 0.4)
-                        (xy 0.6 1)
-                    )
-                    (width 0)
-                    (fill yes)
-                )
-            )
-        )
+        (pad "21" smd rect (at -1 2.0 270) (size 0.9 1.0) (layers "F.Cu" "F.Mask" "F.Paste") (net 81 "JST1_1"))
+        (pad "31" smd rect (at -1 2.0 270) (size 0.9 1.0) (layers "B.Cu" "B.Mask" "B.Paste") (net 81 "JST1_1"))
+        (pad "22" smd rect (at 1 2.0 270) (size 0.9 1.0) (layers "F.Cu" "F.Mask" "F.Paste") (net 82 "JST1_2"))
+        (pad "32" smd rect (at 1 2.0 270) (size 0.9 1.0) (layers "B.Cu" "B.Mask" "B.Paste") (net 82 "JST1_2"))
+        (pad "1" smd rect (at -1 3.6 270) (size 0.9 1.0) (layers "F.Cu" "F.Mask" "F.Paste") (net 80 "BAT_P"))
+        (pad "1" smd rect (at 1 3.6 270) (size 0.9 1.0) (layers "B.Cu" "B.Mask" "B.Paste") (net 80 "BAT_P"))
+        (pad "2" smd rect (at -1 3.6 270) (size 0.9 1.0) (layers "B.Cu" "B.Mask" "B.Paste") (net 3 "GND"))
+        (pad "2" smd rect (at 1 3.6 270) (size 0.9 1.0) (layers "F.Cu" "F.Mask" "F.Paste") (net 3 "GND"))
     )
-    (segment (start 259.4184523 127.62352920000001) (end 257.6184523 127.62352920000001) (width 0.25) (layer "F.Cu") (net 81))
-    (segment (start 259.4184523 127.62352920000001) (end 257.6184523 127.62352920000001) (width 0.25) (layer "B.Cu") (net 81))
-    (segment (start 259.4184523 125.62352920000001) (end 257.6184523 125.62352920000001) (width 0.25) (layer "F.Cu") (net 82))
-    (segment (start 259.4184523 125.62352920000001) (end 257.6184523 125.62352920000001) (width 0.25) (layer "B.Cu") (net 82))
+    (segment (start 259.6184523 127.62352920000001) (end 257.6184523 127.62352920000001) (width 0.5) (layer "F.Cu") (net 81))
+    (segment (start 259.6184523 127.62352920000001) (end 257.6184523 127.62352920000001) (width 0.5) (layer "B.Cu") (net 81))
+    (segment (start 259.6184523 125.62352920000001) (end 257.6184523 125.62352920000001) (width 0.5) (layer "F.Cu") (net 82))
+    (segment (start 259.6184523 125.62352920000001) (end 257.6184523 125.62352920000001) (width 0.5) (layer "B.Cu") (net 82))
+    (segment (start 261.2184523 127.62352920000001) (end 261.2184523 126.62352920000001) (width 0.5) (layer "F.Cu") (net 80))
+    (segment (start 261.2184523 125.62352920000001) (end 261.2184523 126.62352920000001) (width 0.5) (layer "B.Cu") (net 80))
+    (via (at 261.2184523 126.62352920000001) (size 0.6) (drill 0.3) (layers "F.Cu" "B.Cu") (net 80))
   (footprint "ceoloide:power_switch_smd_side"
     (layer "F.Cu")

Commit message: moved the keys around as desired
Parts:
- moved D22 8.69 mm to (258.5, 147.8)
- moved D19 8.69 mm to (200.7, 141.1)
- moved D20 8.69 mm to (220.3, 140.0)
- moved D21 8.69 mm to (239.8, 142.2)
- moved D23 8.69 mm to (215.9, 159.0)
- moved D24 8.69 mm to (235.3, 161.3)
- moved H4 8.69 mm to (260.3, 163.1)
- moved S19 8.69 mm to (208.7, 136.6)
- moved S20 8.69 mm to (229.0, 136.8)
- moved S21 8.69 mm to (248.8, 140.6)
- moved S22 8.69 mm to (267.7, 147.8)
- moved S23 8.69 mm to (224.5, 155.9)
- moved S24 8.69 mm to (244.4, 159.7)
- moved D10 8.48 mm to (195.4, 115.9)
- moved D11 8.48 mm to (194.2, 99.0)
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Other:
- board size 155.7 x 107.9 mm -> 157.7 x 107.7 mm

Commit message: moved components
Parts:
- moved PWR1 3.60 mm to (281.2, 121.7)
- moved RST1 3.60 mm to (281.2, 131.9)
- moved JST1 3.60 mm to (259.6, 121.7)
- moved DISP1 3.60 mm to (268.6, 95.1)
- moved H5 3.60 mm to (280.6, 75.3)
- moved MCU1 3.60 mm to (268.6, 91.1)
- moved H3 1.80 mm to (214.9, 69.7)
