File: kicad/v2.kicad_pcb (KiCad board)
At the start: 2 copper layers, 157.7 x 107.7 mm, 58 parts

Commit message: looking pretty good so far
Routing:
- net RAW: track 9.83 -> 79.9 mm, vias 0 -> 1
- net RST: track 20.3 -> 81.6 mm
- net VCC: track 9.83 -> 55.1 mm
- net CS: track 9.84 -> 39.5 mm, vias 0 -> 1
- net MOSI: track 9.84 -> 34.8 mm, vias 0 -> 1
- net BAT_P: track 2.00 -> 22.1 mm, vias 1 -> 2
- net SCK: track 9.84 -> 26.7 mm, vias 0 -> 1
- net GND: vias 0 -> 1
- added copper zone on B.Cu, net GND
- added copper zone on F.Cu, net GND

Commit message: on to DRC
Routing:
- net P14: track 158.9 -> 232.5 mm, vias 4 -> 6
- net P9: track 126.4 -> 198.5 mm, vias 4 -> 5
- net P8: track 167.1 -> 237.7 mm, vias 4 -> 7
- net P15: track 117.8 -> 178.6 mm
- net P10: track 136.0 -> 182.7 mm, vias 4 -> 5
- net P16: track 122.8 -> 152.5 mm
- net CS: track 39.5 -> 46.3 mm
- net VCC: track 55.1 -> 51.7 mm, vias 0 -> 1
- net RST: track 81.6 -> 79.6 mm, vias 1 -> 2
- net GND: vias 1 -> 27

Commit message: done?
Routing:
- net GND: vias 27 -> 26
Changed lines of the file:
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@@
 	)
 	(via
-		(at 258.5 74.5)
-		(size 0.8)
-		(drill 0.4)
-		(layers "F.Cu" "B.Cu")
-		(free yes)
-		(net 3)
-	)
-	(via
 		(at 266 74)
 		(size 0.8)
@@
 	)
 	(segment
+		(start 216.468956 125.5)
+		(end 211.57695 130.392006)
+		(width 0.25)
+		(layer "F.Cu")
+		(net 6)
+	)
+	(segment
 		(start 211.57695 130.392007)
 		(end 209.651749 132.606697)
@@
 	)
 	(segment
-		(start 167.38813 140.982874)
-		(end 166.234616 141.313639)
-		(width 0.2)
+		(start 252 124)
+		(end 250.5 125.5)
+		(width 0.25)
 		(layer "F.Cu")
 		(net 6)
 	)
 	(segment
-		(start 216.968956 125)
-		(end 211.57695 130.392006)
-		(width 0.25)
+		(start 167.38813 140.982874)
+		(end 166.234616 141.313639)
+		(width 0.2)
 		(layer "F.Cu")
 		(net 6)
@@
 	)
 	(segment
-		(start 251 125)
-		(end 250.5 125)
-		(width 0.25)
-		(layer "F.Cu")
-		(net 6)
-	)
-	(segment
-		(start 252 124)
-		(end 251 125)
-		(width 0.25)
-		(layer "F.Cu")
-		(net 6)
-	)
-	(segment
-		(start 251 125)
-		(end 216.968956 125)
+		(start 250.5 125.5)
+		(end 216.468956 125.5)
 		(width 0.25)
 		(layer "F.Cu")
@@
 	)
 	(segment
+		(start 265.176685 105.748451)
+		(end 265.176685 106.385901)
+		(width 0.25)
+		(layer "B.Cu")
+		(net 6)
+	)
+	(segment
 		(start 165.081102 141.644403)
 		(end 166.234616 141.313639)
@@
 	)
 	(segment
-		(start 264.37837 105.021901)
-		(end 265.176685 105.820216)
+		(start 260.657569 105.021901)
+		(end 264.450135 105.021901)
 		(width 0.25)
 		(layer "B.Cu")
@@
 	)
 	(segment
-		(start 265.176685 105.820216)
-		(end 265.176685 106.385901)
-		(width 0.25)
-		(layer "B.Cu")
-		(net 6)
-	)
-	(segment
 		(start 271.616089 105)
 		(end 266.562586 105)
@@
 	)
 	(segment
-		(start 259.780685 105.898785)
-		(end 260.657569 105.021901)
-		(width 0.25)
-		(layer "B.Cu")
-		(net 6)
-	)
-	(segment
 		(start 162.514537 135.014537)
 		(end 162.514537 140.221733)
@@
 	)
 	(segment
+		(start 259.780685 105.898785)
+		(end 260.657569 105.021901)
+		(width 0.25)
+		(layer "B.Cu")
+		(net 6)
+	)
+	(segment
 		(start 154.193883 108.589851)
 		(end 154.193883 114.693883)
@@
 	)
 	(segment
+		(start 264.450135 105.021901)
+		(end 265.176685 105.748451)
+		(width 0.25)
+		(layer "B.Cu")
+		(net 6)
+	)
+	(segment
 		(start 205.042905 130.848912)
 		(end 207.257595 132.774112)
@@
 	)
 	(segment
-		(start 252 124)
-		(end 259.780685 116.219315)
+		(start 273.00199 106.385901)
+		(end 271.616089 105)
 		(width 0.25)
 		(layer "B.Cu")
@@
 	)
 	(segment
-		(start 273.00199 106.385901)
-		(end 271.616089 105)
+		(start 259.780685 116.219315)
+		(end 259.780685 105.898785)
 		(width 0.25)
 		(layer "B.Cu")
@@
 	)
 	(segment
-		(start 259.780685 116.219315)
-		(end 259.780685 105.898785)
-		(width 0.25)
-		(layer "B.Cu")
-		(net 6)
-	)
-	(segment
 		(start 166.85957 135)
 		(end 194.5 135)
@@
 	)
 	(segment
-		(start 260.657569 105.021901)
-		(end 264.37837 105.021901)
+		(start 162.514537 140.221733)
+		(end 162.514537 139.345033)
 		(width 0.25)
 		(layer "B.Cu")
@@
 	)
 	(segment
-		(start 162.514537 140.221733)
-		(end 162.514537 139.345033)
+		(start 252 124)
+		(end 259.780685 116.219315)
 		(width 0.25)
 		(layer "B.Cu")
@@
 	)
 	(segment
+		(start 251 127)
+		(end 242 127)
+		(width 0.25)
+		(layer "F.Cu")
+		(net 10)
+	)
+	(segment
 		(start 232.833459 131.270459)
 		(end 230.55293 133.117195)
@@
 	)
 	(segment
-		(start 253 124.951)
-		(end 253 125)
+		(start 242 127)
+		(end 237.729541 131.270459)
 		(width 0.25)
 		(layer "F.Cu")
@@
 	)
 	(segment
-		(start 237.152919 126.951)
-		(end 232.83346 131.270459)
+		(start 253 124.951)
+		(end 253 125)
 		(width 0.25)
 		(layer "F.Cu")
@@
 	)
 	(segment
-		(start 251.049 126.951)
-		(end 237.152919 126.951)
-		(width 0.25)
-		(layer "F.Cu")
-		(net 10)
-	)
-	(segment
 		(start 180.594707 81.092166)
 		(end 178.828685 83.435756)
@@
 	)
 	(segment
-		(start 253 125)
-		(end 251.049 126.951)
+		(start 237.729541 131.270459)
+		(end 232.83346 131.270459)
 		(width 0.25)
 		(layer "F.Cu")
@@
 		(net 10)
 	)
+	(segment
+		(start 253 125)
+		(end 251 127)
+		(width 0.25)
+		(layer "F.Cu")
+		(net 10)
+	)
 	(via
 		(at 229.359504 132.991761)
@@
 	)
 	(segment
-		(start 263.176685 122.745901)
-		(end 263.176685 121.745901)
+		(start 277 124)
+		(end 279.437586 124)
 		(width 0.5)
 		(layer "F.Cu")
@@
 	)
 	(segment
-		(start 277 124)
-		(end 279.437586 124)
+		(start 264 122.745901)
+		(end 263.176685 122.745901)
 		(width 0.5)
 		(layer "F.Cu")
@@
 		(net 75)
 	)
+	(segment
+		(start 265 121.745901)
+		(end 264 122.745901)
+		(width 0.5)
+		(layer "F.Cu")
+		(net 75)
+	)
 	(via
 		(at 277 124)
@@
 	)
 	(via
-		(at 263.176685 121.745901)
+		(at 265 121.745901)
 		(size 0.8)
 		(drill 0.4)
@@
 	)
 	(segment
-		(start 268.745901 120.745901)
+		(start 269.745901 121.745901)
 		(end 271.995901 123.995901)
 		(width 0.5)
@@
 	)
 	(segment
-		(start 263.176685 120.745901)
-		(end 263.176685 121.745901)
+		(start 264 120.745901)
+		(end 263.176685 120.745901)
 		(width 0.5)
 		(layer "B.Cu")
@@
 	)
 	(segment
-		(start 277 124)
-		(end 279.437586 124)
+		(start 265 121.745901)
+		(end 269.745901 121.745901)
+		(width 0.5)
+		(layer "B.Cu")
+		(net 75)
+	)
+	(segment
+		(start 265 121.745901)
+		(end 264 120.745901)
 		(width 0.5)
 		(layer "B.Cu")
@@
 	)
 	(segment
-		(start 263.176685 120.745901)
-		(end 268.745901 120.745901)
+		(start 277 124)
+		(end 279.437586 124)
 		(width 0.5)
 		(layer "B.Cu")

Commit message: minor
Routing:
- net GND: vias 26 -> 27
Changed lines of the file:
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@@
 	)
 	(via
-		(at 266 74)
+		(at 265 74)
 		(size 0.8)
 		(drill 0.4)
@@
 	)
 	(via
-		(at 271 74)
+		(at 272.5 74)
 		(size 0.8)
 		(drill 0.4)
@@
 		(size 0.8)
 		(drill 0.4)
+		(layers "F.Cu" "B.Cu")
+		(free yes)
+		(net 3)
+	)
+	(via
+		(at 279.5 95)
+		(size 0.8)
+		(drill 0.4)
