File: kicad/board.kicad_pcb (KiCad board)
At the start: 2 copper layers, 157.7 x 107.7 mm, 58 parts

Commit message: generated gerbers
Other:
- board text added: "Isaac Olson"
- board text added: "qwerky v1.0"
Changed lines of the file:
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@@
 			(outputformat 1)
 			(mirror no)
-			(drillshape 1)
+			(drillshape 0)
 			(scaleselection 1)
-			(outputdirectory "")
+			(outputdirectory "qwerky-gerbers/")
 		)
 	)
@@
 		(layer "Edge.Cuts")
 	)
+	(gr_text "qwerky v1.0"
+		(at 257.5 128.5 0)
+		(layer "F.SilkS")
+		(effects
+			(font
+				(size 1.5 1.5)
+				(thickness 0.3)
+				(bold yes)
+			)
+			(justify left bottom)
+		)
+	)
+	(gr_text "Isaac Olson"
+		(at 257.5 131.5 0)
+		(layer "F.SilkS")
+		(effects
+			(font
+				(size 1.5 1.5)
+				(thickness 0.3)
+				(bold yes)
+			)
+			(justify left bottom)
+		)
+	)
+	(gr_text "qwerky v1.0"
+		(at 271 128.5 0)
+		(layer "B.SilkS")
+		(effects
+			(font
+				(size 1.5 1.5)
+				(thickness 0.3)
+				(bold yes)
+			)
+			(justify left bottom mirror)
+		)
+	)
+	(gr_text "Isaac Olson"
+		(at 271 131.5 0)
+		(layer "B.SilkS")
+		(effects
+			(font
+				(size 1.5 1.5)
+				(thickness 0.3)
+				(bold yes)
+			)
+			(justify left bottom mirror)
+		)
+	)
 	(segment
 		(start 142.13642 110.694883)
@@
 	)
 	(via
-		(at 269.5 131.5)
+		(at 271 135)
 		(size 0.8)
 		(drill 0.4)
